File: Kicad project/two_lipol_charger.kicad_pcb (KiCad board)
At the start: 2 copper layers, 71.1 x 40.6 mm, 66 parts, among them J1 Conn_01x18, SW1 SW_DPDT_x2, SW2 SW_DPDT_x2, SW3 SW_DIP_x04, U1 FAN9673, U2 LM358D

Commit message: Version 1.0
Parts:
- C31, C32, C33, C41, C47, C48, C49, C50, C55, C56, C57, C58, C59, C60, C62, R57, R63, R64, R73: moved to B.Cu
- moved C59 106.5 mm to (71.1, 97.0), turned to 90 degrees
- moved C63 99.5 mm to (65.8, 98.4), turned to 180 degrees
- moved C60 98.4 mm to (68.6, 97.0), turned to 90 degrees
- moved R73 97.5 mm to (78.8, 74.7), turned to 90 degrees
- moved C57 91.7 mm to (78.7, 97.0), turned to 90 degrees
- moved C56 90.7 mm to (83.8, 97.0), turned to 90 degrees
- moved C58 90.6 mm to (76.2, 97.0), turned to 90 degrees
- moved C48 87.5 mm to (71.8, 86.6), turned to 180 degrees
- moved R63 86.5 mm to (75.1, 85.3), turned to 270 degrees
- moved C32 86.1 mm to (99.1, 93.0), turned to 270 degrees
- moved C49 84.8 mm to (71.8, 89.2), turned to 180 degrees
- moved R64 84.3 mm to (75.1, 90.4), turned to 270 degrees
- moved C62 83.0 mm to (76.2, 74.7), turned to 270 degrees
- moved C47 82.6 mm to (71.8, 84.1), turned to 180 degrees
- moved C64 78.0 mm to (81.5, 75.9), turned to 270 degrees
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Connections:
- net Net-(C43-Pad1) renamed VLPK
- J1 pad 18: 12v -> 12V
Routing:
- net GND: track 0.00 -> 180.9 mm, vias 0 -> 11
- net FBPFC: track 0.00 -> 149.8 mm, vias 0 -> 1
- net PVO: track 0.00 -> 62.3 mm, vias 0 -> 2
- net IAC: track 0.00 -> 43.2 mm
- net RDY: track 0.00 -> 43.1 mm, vias 0 -> 1
- net CVM2: track 0.00 -> 41.5 mm
- net BIBO: track 0.00 -> 39.1 mm
- net 15V: track 0.00 -> 33.1 mm, vias 0 -> 2
- net 12V: track 0.00 -> 27.1 mm, vias 0 -> 1
- net CVM3: track 0.00 -> 24.5 mm
- net OPFC1: track 0.00 -> 21.8 mm
- net OPFC2: track 0.00 -> 19.6 mm
- net CS1+: track 0.00 -> 18.8 mm
- net Net-(C61-Pad1): track 0.00 -> 18.7 mm
- net Net-(C39-Pad2): track 0.00 -> 18.7 mm
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- added copper zone on B.Cu, net GND
Other:
- board size 71.1 x 40.6 mm -> 71.1 x 40.8 mm
- net class Default: trace_width 0.25 -> 0.8
- board text added: "12V"
- board text added: "A"
- board text added: "A: CH2 EN B: CH3 EN C: VR to PVO D: 12V to VR"
- board text added: "B"
- board text added: "BIBO"
- board text added: "C"
- board text added: "D"
- board text added: "EN2"
- board text added: "EN3"
- board text added: "FAN9673 Daughter Card rkradim@yandex.ru TotalRace"
- board text added: "G1"
- board text added: "G2"
- board text added: "G3"
- board text added: "IAC"
- board text added: "PVO"
- board text added: "RDY"
- board text added: "SW2"
- board text added: "SW2/3 : Channel Man. off SW2/3 : Channel Man. on"
- board text added: "SW3"
- board text added: "VLPK"
- board text added: "VR: 0V <---> 3.5V"
- board text added: "fbpfc"
