File: Kicad project/two_lipol_charger.sch (KiCad schematic (older format))
At the start: 66 parts, among them J1 Conn_01x18, SW1 SW_DPDT_x2, SW2 SW_DPDT_x2, SW3 SW_DIP_x04, U1 FAN9673, U2 LM358D

Commit message: Version 1.0
Connections:
- net labels added: VLPK
- net labels removed: 12v
- wire segments 311 -> 313
Changed lines of the file:
@@
 FBPFC
 Text GLabel 1800 2650 2    50   Input ~ 0
-12v
+12V
 $Comp
 L power:GND #PWR0101
@@
 	3850 4200 3850 4350
 Wire Wire Line
-	4350 4000 4600 4000
-Wire Wire Line
-	4600 4000 4600 3850
-Wire Wire Line
-	4600 3850 5400 3850
+	4350 4000 4450 4000
+Wire Wire Line
+	4450 4000 4450 3850
+Wire Wire Line
+	4450 3850 5400 3850
 Connection ~ 4350 4000
 $Comp
@@
 Connection ~ 3250 4450
 Wire Wire Line
-	3750 4650 4700 4650
-Wire Wire Line
-	4700 4650 4700 3950
-Wire Wire Line
-	4700 3950 5400 3950
+	3750 4650 4500 4650
+Wire Wire Line
+	4500 4650 4500 3950
+Wire Wire Line
+	4500 3950 5400 3950
 Connection ~ 3750 4650
 Wire Wire Line
@@
 $EndComp
 Wire Wire Line
-	4900 4050 4900 4250
+	4900 4050 4900 4150
 $Comp
 L power:GND #PWR0109
@@
 Wire Wire Line
 	13400 4550 13400 4450
+Text GLabel 4850 4150 0    50   Input ~ 0
+VLPK
+Wire Wire Line
+	4850 4150 4900 4150
+Connection ~ 4900 4150
+Wire Wire Line
+	4900 4150 4900 4250
 $EndSCHEMATC
